Commit message: add camera

File: rotors_description/urdf/ardrone_base.xacro (robot description, xacro)
@@ -80,4 +80,14 @@
     </xacro:odometry_plugin_macro>
   </xacro:if>
+  <!-- Forward facing camera -->
+    <xacro:include filename="$(find rotors_description)/urdf/generic_camera.urdf.xacro" />
+    <xacro:generic_camera name="front_cam" parent="base_link" ros_topic="camera/image" cam_info_topic="camera/camera_info" update_rate="20" res_x="640" res_y="480" image_format="R8G8B8" hfov="90">
+      <origin xyz="0.05 0.0 -0.06" rpy="0 0 0"/>
+    </xacro:generic_camera>
+    <!-- Downward facing camera -->
+    <xacro:include filename="$(find rotors_description)/urdf/generic_camera.urdf.xacro" />
+    <xacro:generic_camera name="downward_cam" parent="base_link" ros_topic="camera/image" cam_info_topic="camera/camera_info" update_rate="20" res_x="640" res_y="480" image_format="L8" hfov="100">
+      <origin xyz="0.4 0.0 -0.0" rpy="0 ${M_PI/2} 0"/>
+    </xacro:generic_camera>
   <xacro:if value="$(arg enable_logging)">
     <!-- Instantiate a logger -->

Commit message: add husky package to rotors

File: rotors_description/urdf/ardrone_base.xacro (robot description, xacro)
@@ -89,3 +89,8 @@
     </xacro:bag_plugin_macro>
   </xacro:if>
+  <!-- 45 Degree Down-forward facing camera -->
+  <xacro:include filename="$(find rotors_description)/urdf/generic_camera.urdf.xacro" />
+  <xacro:generic_camera name="front_cam" parent="base_link" ros_topic="camera/image" cam_info_topic="camera/camera_info" update_rate="10" res_x="320" res_y="240" image_format="R8G8B8" hfov="90">
+  <origin xyz="0.05 0.0 -0.06" rpy="0 ${M_PI/4} 0"/>
+  </xacro:generic_camera>
 </robot>

Commit message: modify launch file

File: rotors_description/urdf/ardrone_base.xacro (robot description, xacro)
@@ -87,6 +87,6 @@
     <!-- Downward facing camera -->
     <xacro:include filename="$(find rotors_description)/urdf/generic_camera.urdf.xacro" />
-    <xacro:generic_camera name="downward_cam" parent="base_link" ros_topic="camera/image" cam_info_topic="camera/camera_info" update_rate="20" res_x="640" res_y="480" image_format="L8" hfov="100">
-      <origin xyz="0.4 0.0 -0.0" rpy="0 ${M_PI/2} 0"/>
+    <xacro:generic_camera name="downward_cam" parent="base_link" ros_topic="camera/image" cam_info_topic="camera/camera_info" update_rate="20" res_x="1280" res_y="960" image_format="R8G8B8" hfov="60">
+      <origin xyz="0.00 0.0 -0.06" rpy="0 ${M_PI/2} 0"/>
     </xacro:generic_camera>
   <xacro:if value="$(arg enable_logging)">
