Commit message: add apriltag from sketchup and reverse

File: husky_description/urdf/decorations.urdf.xacro (robot description, xacro)
@@ -111,5 +111,5 @@
           <origin xyz="0 0 0" rpy="0 0 0" />
           <geometry>
-            <mesh filename="package://husky_description/meshes/top_plate_texture.dae" />
+            <mesh filename="package://husky_description/meshes/top_plate_texture2.dae" />
           </geometry>
         </visual>
@@ -118,5 +118,5 @@
         <parent link="base_link" />
         <child link="top_plate_texture_link"/>
-        <origin xyz="-0.1 0.6 -0.330" rpy="1.57 0 0"/>
+        <origin xyz="-0.1 0.6 -0.430" rpy="1.57 0 0"/>
       </joint>
     </xacro:if>
